File: hub_2.kicad_sch (KiCad schematic)
At the start: 51 parts, among them J7 USB_C_Receptacle_USB2.0_16P, J8 USB_C_Receptacle_USB2.0_16P, J9 Header 01x04 0.1", U10 USB2514B-I/M2, U11 MIC2026-1xM, U12 MIC2026-1xM, U7 USBLC6-2P6, U8 USBLC6-2P6, U9 USBLC6-2P6, Y1 24MHz

Commit message: Finished Camera Hub
Parts:
- removed FB6: 600R, Inductor_SMD:L_0603_1608Metric, symbol Device:FerriteBead_Small
- removed J9: Header 01x04 0.1", Connector_PinHeader_2.54mm:PinHeader_1x04_P2.54mm_Vertical, symbol Connector_Generic:Conn_01x04
- added C20: 100uF, Capacitor_SMD:C_0805_2012Metric, symbol Device:C_Small
- added C21: 0.1uF, Capacitor_SMD:C_0603_1608Metric, symbol Device:C_Small
- added D1: Green, LED_SMD:LED_0603_1608Metric, symbol Device:LED_Small
- added FB1, FB3: 600R, Inductor_SMD:L_0603_1608Metric, symbol Device:FerriteBead_Small
- added FL1: 744230900, CameraHub:CHIP_230900_WRE, symbol Filter:Choke_Wurth_WE-CNSW_744232090
- added J2, J4: USB_C_Receptacle_USB2.0_16P, CameraHub:USBC-121SMT-4BS2S, symbol Connector:USB_C_Receptacle_USB2.0_16P
- added R8: 330R, Resistor_SMD:R_0603_1608Metric, symbol Device:R_Small
- added R9: 10K, Resistor_SMD:R_0603_1608Metric, symbol Device:R_Small
- added U1: USBLC6-2P6, Package_TO_SOT_SMD:SOT-23-6, symbol Power_Protection:USBLC6-2P6
Connections:
- net +3.3V: now also R9.1
- net D3_N: now also J2.A7 (D-), J2.B7 (D-)
- net D3_P: now also J2.A6 (D+), J2.B6 (D+)
- net GND: now also C20.2, C21.2, D1.1 (K), J2.A1 (GND), J2.A12 (GND), J2.B1 (GND), J2.B12 (GND), J2.S1 (SHIELD), J4.A1 (GND), J4.A12 (GND), J4.B1 (GND), J4.B12 (GND), J4.S1 (SHIELD), U1.2 (GND)
- net VBUS3: now also FB1.1
- net VBUS_CONN3: now also FB1.2, J2.A4 (VBUS), J2.A9 (VBUS), J2.B4 (VBUS), J2.B9 (VBUS)
- net PWR4: now reaches U10.20 (PRTPWR4/BC_EN4)
- net PWR4: now also U12.4 (ENB)
- net nOCS4: now reaches U10.21 (OCS_N4)
- net nOCS4: now also U12.3 (FLGB), R9.2
- net HD4_N: now reaches U10.8 (USBDM_DN4/PRT_DIS_M4)
- net HD4_N: now also FL1.4
- net HD4_P: now reaches U10.9 (USBDP_DN4/PRT_DIS_P4)
- net HD4_P: now also FL1.1
- net VBUS4: now reaches U12.5 (OUTB)
- net VBUS4: now also C20.1, C21.1, FB3.1
- new net: D1.2 (A), R8.2
- new net D4_N: J4.A7 (D-), J4.B7 (D-), U1.4 (I/O2)
- new net D4_P: J4.A6 (D+), J4.B6 (D+), U1.6 (I/O1)
- new net FD4_N: FL1.3, U1.3 (I/O2)
- new net FD4_P: FL1.2, U1.1 (I/O1)
- new net VBUS_CONN4: FB3.2, J4.A4 (VBUS), J4.A9 (VBUS), J4.B4 (VBUS), J4.B9 (VBUS), R8.1, U1.5 (VBUS)
- no-connect marks 18 -> 19
Other:
- moved on the sheet: C12, C13, C14, C15, C16, C17, C18, C19, D4, D5, D6, R11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
